File: Layout/v1/early-bird.brd (EAGLE design)
At the start: 98.5 x 80.8 mm, 28 parts, among them U1 ATMEGA328P-AU

Commit message: Add PCB progress.
Parts:
- added C11, C16, C22: 1uF, resistor:C0603
- added C12, C17, C18, C21: 100n, resistor:C0402
- added C13: 10uF, resistor:C1210
- added C14, C15: 22p, resistor:C0402
- added C19: 33n, resistor:C0402
- added C20: (no value), resistor:C0402
- added D1: MBRA340T3, diode:SMA
- added J1: 22-27-2021-02, con-molex:6410-02
- added J2: AVR_SPI_PRG_62X3_LOCK, SparkFun-Connectors:2X3_LOCK
- added JP1: M02PTH, SparkFun-Connectors:1X02
- added LED4: (no value), led:CHIPLED_1206
- added R10, R7, R8, R9: 10, resistor:R0402
- added R11, R12, R13, R14: (no value), resistor:R0402
- added U$10: MULTICOMP_8MM_INDUCTOR, Ava:8MM_SQ_INDUCTOR
- added U$7: ABRACON_ABM3_CRYSTAL, Ava:ABRACON_ABM3_CRYSTAL
- added U$8: ADP1612, Ava:SOP65P490X110-8N
- added U$9: BGM1034N7, Ava:TSNP-7-10
- C9: value 100n -> 10uF; device resistor:C0402 -> resistor:C1210
- U$1, U$2: value KEYSTONE-82-AAA-BATTERY-HOLDER -> KEYSTONE-92-AA-BATTERY-HOLDER; device Ava:KEYSTONE-82-AAA-BATTERY -> Ava:KEYSTONE-92-AA-BATTERY
- moved C9 77.7 mm to (72.5, 11.0), turned to 270 degrees
- moved R1 45.3 mm to (61.5, 12.5), turned to 180 degrees
- moved C6 35.6 mm to (87.5, 45.5)
- moved C2 30.1 mm to (87.5, 44.0), turned to 0 degrees
- moved R2 29.8 mm to (73.0, 38.5), turned to 270 degrees
- moved R3 27.9 mm to (73.0, 42.5), turned to 270 degrees
- moved C8 27.0 mm to (71.0, 42.5), turned to 90 degrees
- moved C1 25.9 mm to (71.0, 38.5), turned to 90 degrees
- moved U$1 19.8 mm to (66.5, 55.8)
- moved C4 16.4 mm to (51.0, 20.5), turned to 180 degrees
- moved C7 16.0 mm to (51.0, 19.0), turned to 180 degrees
- moved U1 14.4 mm to (63.3, 38.4)
- moved R4 11.0 mm to (12.0, 69.0)
- moved C10 10.5 mm to (8.50, 68.5), turned to 90 degrees
- moved R5 10.5 mm to (25.5, 61.0)
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Connections:
- removed net +: C2.1, C3.1, C4.1, C5.1, C6.1, C7.1, R1.2, R2.2, R4.1, U$1.VBATT, U$1.VBATT1, U$2.VBATT, U$2.VBATT1, U$4.VCC, U$5.6_V_BCKP, U$5.7_VCC_IO, U$5.8_VCC, U1.18, U1.4, U1.6
- removed net -: C1.2, C10.2, C2.2, C3.2, C4.2, C5.2, C6.2, C7.2, C8.2, C9.2, LED1.C, LED2.C, LED3.C, R3.1, U$1.GND, U$1.GND2, U$2.GND, U$2.GND2, U$4.GND1, U$4.GND2, U$4.GND3, U$5.10_GND, U$5.12_GND, U$5.1_GND, U$6.2, U$6.3, U$6.4, U$6.5, U1.21, U1.3, U1.5
- removed net N$9: U$4.DIO0
- new net AUX+: C11.1, C12.1, C13.1, D1.C, J1.1, R10.1, R13.2
- new net BATT+: C16.1, C17.1, C18.1, C2.1, C21.1, C22.1, C3.1, C4.1, C5.1, C6.1, C7.1, C9.1, J2.2, JP1.1, JP1.2, R1.2, R14.2, R2.2, R4.1, U$1.VBATT, U$1.VBATT1, U$10.P$2, U$4.VCC, U$5.6_V_BCKP, U$5.7_VCC_IO, U$5.8_VCC, U$8.3, U$8.6, U1.18, U1.4, U1.6
- new net BATT-: C1.2, C10.2, C11.2, C12.2, C13.2, C14.2, C15.2, C16.2, C17.2, C18.2, C19.2, C2.2, C20.1, C21.2, C22.2, C3.2, C4.2, C5.2, C6.2, C7.2, C8.2, C9.2, J1.2, J2.6, L1.2, LED1.C, LED2.C, LED3.C, LED4.C, R12.1, R14.1, R3.1, U$2.GND, U$2.GND2, U$4.GND1, U$4.GND2, U$4.GND3, U$5.10_GND, U$5.12_GND, U$5.1_GND, U$6.2, U$6.3, U$6.4, U$6.5, U$8.4, U$8.7, U$9.GND, U1.21, U1.3, U1.5
- new net DIO0: U$4.DIO0, U1.11
- new net DIO1: U$4.DIO1, U1.12
- new net DIO2: U$4.DIO2, U1.13
- new net LNA+: C10.1, R4.2, U$9.PON, U$9.VCC
- new net N$10: R7.1, U1.32
- new net N$12: R8.1, U1.1
- new net N$13: R9.1, U1.2
- new net N$14: LED1.A, R9.2
- new net N$15: LED4.A, R10.2
- new net N$16: U$1.GND, U$1.GND2, U$2.VBATT, U$2.VBATT1
- new net N$17: C15.1, U$7.P$2, U1.8
- new net N$18: C14.1, U$7.P$1, U1.7
- new net N$19: C19.1, U$8.8
- new net N$20: R11.2, U$8.1
- new net N$21: R12.2, R13.1, U$8.2
- new net N$23: D1.A, U$10.P$1, U$8.5
- new net N$24: L2.2, U$9.AI
- new net N$25: U$5.11_RF_IN, U$9.RFOUT
- net MISO: now also J2.1
- net MOSI: now also J2.4
- net N$11: now also L2.1, U$9.SO; no longer C10.1, C9.1, R4.2
- net N$2: now also L1.1, U$9.RFIN; no longer U$5.11_RF_IN
- net N$3: now also LED3.A, R7.2; no longer LED1.A, U1.32
- net N$4: now also R8.2; no longer U1.1
- net N$5: now also C20.2, R11.1; no longer LED3.A, U1.2
- net RESET: now also J2.5
- net SCK: now also J2.3
Routing:
- net BATT+: track 0.00 -> 251.3 mm, vias 0 -> 2
- net N$14: track 0.00 -> 78.4 mm
- net N$4: track 15.9 -> 70.5 mm
- net GPS_RX: track 0.00 -> 53.5 mm
- net GPS_TX: track 0.00 -> 53.4 mm, vias 0 -> 2
- net MISO: track 0.00 -> 50.4 mm, vias 0 -> 2
- net RESET: track 0.00 -> 43.5 mm, vias 0 -> 4
- net MOSI: track 0.00 -> 38.2 mm, vias 0 -> 2
- net BATT-: track 0.00 -> 34.4 mm, vias 0 -> 129
- net N$3: track 21.9 -> 52.7 mm
- net SS: track 0.00 -> 29.6 mm, vias 0 -> 2
- net SCK: track 0.00 -> 26.7 mm
- net DIO2: track 0.00 -> 26.3 mm, vias 0 -> 2
- net DIO1: track 0.00 -> 23.7 mm, vias 0 -> 2
- net +: track 21.9 -> 0.00 mm
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- added copper zone on layer 1, net AUX+
- added copper zone on layer 1, net BATT+
- added copper zone on layer 1, net BATT-
- added copper zone on layer 16, net BATT-
- added copper zone on layer 1, net N$16
- added copper zone on layer 1, net N$23
- removed copper zone on layer 1, net +
- removed copper zone on layer 1, net -
- removed copper zone on layer 16, net -
Other:
- board text added: "AUX ON"
- board text added: "Phil M0DNY - 2014"
- board text added: "https://www.philcrump.co.uk/"

Commit message: Layout Progress, redraw schematic a little.
Parts:
- added C23: 10uF, resistor:C1210
- moved C16 2.25 mm to (87.5, 40.2)
- moved C17 2.25 mm to (87.5, 38.8)
- moved C2 2.25 mm to (87.5, 41.8)
- moved C6 2.25 mm to (87.5, 43.2)
- moved J2 2.25 mm to (79.0, 27.8)
- moved R12 2.14 mm to (69.5, 2.00), turned to 180 degrees
- moved R7 0.75 mm to (55.0, 44.8)
- moved R8 0.50 mm to (55.0, 43.5)
- moved C20 0.25 mm to (79.2, 2.00)
- moved C21 0.25 mm to (72.8, 2.00)
- moved R11 0.25 mm to (81.5, 3.00)
- moved R13 0.25 mm to (68.5, 3.25)
- moved R9 0.25 mm to (55.0, 42.2)
Connections:
- new net N$9: JP1.1, R14.2, U$8.3
- net BATT+: now also C23.1; no longer JP1.1, R14.2, U$8.3
- net BATT-: now also C23.2
Routing:
- net BATT+: track 251.3 -> 232.4 mm
- net N$9: track 0.00 -> 11.7 mm
- net RESET: track 43.5 -> 39.7 mm
- net SCK: track 26.7 -> 29.0 mm
- net BATT-: track 34.4 -> 32.1 mm, vias 129 -> 132
- net MOSI: track 38.2 -> 39.8 mm
- net N$21: track 13.0 -> 12.2 mm
- net N$3: track 52.7 -> 52.0 mm
- net N$10: track 7.74 -> 6.99 mm
- net N$4: track 70.5 -> 69.8 mm
- net AUX+: track 14.8 -> 14.1 mm
- net N$12: track 6.24 -> 5.74 mm
Other:
- board text added: "10u"
- board text added: "1u"

Commit message: Stage for fab?
Parts:
- added PAD1, PAD2: (no value), wirepad:SMD1,27-2,54
- added Q1: (no value), crystal:CTS406
- moved R10 8.81 mm to (49.2, 2.50)
Connections:
- new net N$22: PAD1.1, Q1.1
- new net N$26: PAD2.1, Q1.3
- net BATT-: now also Q1.2, Q1.4
Routing:
- net N$22: track 0.00 -> 4.90 mm
- net N$26: track 0.00 -> 4.11 mm
- net AUX+: track 14.1 -> 17.2 mm
- net N$15: track 13.8 -> 14.8 mm
- net BATT-: vias 132 -> 142
Other:
- board text added: ".1u"
- board text added: "10K"
- board text added: "10R"
- board text added: "150R"
- board text added: "22K"
- board text added: "22p"
- board text added: "33n"
- board text added: "3n3"
- board text added: "3x 47R"
- board text added: "6K8"
- board text added: "8.2nH"
- board text added: "9.1nH"
- board text added: "L3"
- board text added: "X1"
- board text added: "X2"
