File: Layout/v1/early-bird.brd (EAGLE design)
At the start: 98.5 x 80.8 mm, 61 parts, among them J1 22-27-2021-02, J2 AVR_SPI_PRG_62X3_LOCK, U1 ATMEGA328P-AU

Commit message: More Final tweaks..
Parts:
- moved C16 0.25 mm to (87.2, 40.2)
- moved C17 0.25 mm to (87.2, 38.8)
- moved C2 0.25 mm to (87.2, 41.8)
- moved C6 0.25 mm to (87.2, 43.2)
Routing:
- net BATT-: vias 142 -> 144
Changed lines of the file:
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@@
 <text x="51" y="17.75" size="0.8128" layer="51" font="vector" ratio="15" align="center">1u</text>
 <text x="51" y="21.5" size="0.8128" layer="51" font="vector" ratio="15" align="center">.1u</text>
-<text x="85.5" y="41.75" size="0.8128" layer="51" font="vector" ratio="15" align="center">.1u</text>
-<text x="85.5" y="38.75" size="0.8128" layer="51" font="vector" ratio="15" align="center">.1u</text>
+<text x="85.25" y="41.75" size="0.8128" layer="51" font="vector" ratio="15" align="center">.1u</text>
+<text x="85.25" y="38.75" size="0.8128" layer="51" font="vector" ratio="15" align="center">.1u</text>
 <text x="57" y="41" size="0.8128" layer="51" font="vector" ratio="15" rot="R270" align="center">.1u</text>
-<text x="85.25" y="43.25" size="0.8128" layer="51" font="vector" ratio="15" rot="R180" align="center">1u</text>
-<text x="85.25" y="40.25" size="0.8128" layer="51" font="vector" ratio="15" rot="R180" align="center">1u</text>
+<text x="85" y="43.25" size="0.8128" layer="51" font="vector" ratio="15" rot="R180" align="center">1u</text>
+<text x="85" y="40.25" size="0.8128" layer="51" font="vector" ratio="15" rot="R180" align="center">1u</text>
 <text x="87.5" y="34.5" size="0.8128" layer="51" font="vector" ratio="15" rot="R180" align="center">10u</text>
 <text x="71" y="36.5" size="0.8128" layer="51" font="vector" ratio="15" rot="R270" align="center">.1u</text>
@@
 <text x="9.75" y="69" size="0.8128" layer="51" font="vector" ratio="15" rot="R90" align="center">1u</text>
 <text x="55.25" y="45.75" size="0.8128" layer="51" font="vector" ratio="15" rot="R180" align="center">3x 47R</text>
-<text x="49.25" y="3.5" size="0.8128" layer="51" font="vector" ratio="15" rot="R180" align="center">150R</text>
+<text x="49.25" y="1.5" size="0.8128" layer="51" font="vector" ratio="15" rot="R180" align="center">150R</text>
 <text x="2.25" y="69.75" size="0.8128" layer="51" font="vector" ratio="15" rot="R180" align="center">9.1nH</text>
 <text x="3.25" y="62.25" size="0.8128" layer="51" font="vector" ratio="15" rot="R180" align="center">8.2nH</text>
@@
 <wire x1="58.5" y1="5.5" x2="60" y2="5.5" width="0.4064" layer="51"/>
 <wire x1="59.25" y1="6.25" x2="59.25" y2="4.75" width="0.4064" layer="51"/>
-<text x="83.75" y="10.75" size="0.8128" layer="51" font="vector" ratio="15" rot="R90" align="center">L3</text>
+<text x="83.5" y="11" size="0.8128" layer="51" font="vector" ratio="15" rot="R90" align="center">L3</text>
 <text x="51" y="38" size="0.8128" layer="51" font="vector" ratio="15" rot="R270" align="center">X1</text>
 <text x="80" y="1" size="0.8128" layer="51" font="vector" ratio="15" align="center">3n3</text>
@@
 </element>
 <element name="C1" library="resistor" package="C0402" value="100n" x="71" y="38.5" smashed="yes" rot="R90"/>
-<element name="C2" library="resistor" package="C0402" value="100n" x="87.5" y="41.75" smashed="yes"/>
+<element name="C2" library="resistor" package="C0402" value="100n" x="87.25" y="41.75" smashed="yes"/>
 <element name="C3" library="resistor" package="C0402" value="100n" x="23" y="67" smashed="yes" rot="R90"/>
 <element name="C4" library="resistor" package="C0402" value="100n" x="51" y="20.5" smashed="yes" rot="R180"/>
@@
 </element>
 <element name="C5" library="resistor" package="C0603" value="1uF" x="24.5" y="67" smashed="yes" rot="R90"/>
-<element name="C6" library="resistor" package="C0603" value="1uF" x="87.5" y="43.25" smashed="yes"/>
+<element name="C6" library="resistor" package="C0603" value="1uF" x="87.25" y="43.25" smashed="yes"/>
 <element name="C7" library="resistor" package="C0603" value="1uF" x="51" y="19" smashed="yes" rot="R180"/>
 <element name="C10" library="resistor" package="C0603" value="1uF" x="8.5" y="68.5" smashed="yes" rot="R90"/>
@@
 <element name="J2" library="SparkFun-Connectors" package="2X3_LOCK" value="AVR_SPI_PRG_62X3_LOCK" x="79" y="27.75" smashed="yes" rot="R270"/>
 <element name="U$7" library="Ava" package="ABRACON_ABM3_CRYSTAL" value="ABRACON_ABM3_CRYSTAL" x="53.5" y="36.5" rot="R270"/>
-<element name="C16" library="resistor" package="C0603" value="1uF" x="87.5" y="40.25" smashed="yes"/>
-<element name="C17" library="resistor" package="C0402" value="100n" x="87.5" y="38.75" smashed="yes"/>
+<element name="C16" library="resistor" package="C0603" value="1uF" x="87.25" y="40.25" smashed="yes"/>
+<element name="C17" library="resistor" package="C0402" value="100n" x="87.25" y="38.75" smashed="yes"/>
 <element name="C18" library="resistor" package="C0402" value="100n" x="57" y="39" smashed="yes" rot="R270"/>
 <element name="U$8" library="Ava" package="SOP65P490X110-8N" value="ADP1612" x="77.5" y="4.75" rot="R180"/>
@@
 <via x="91" y="40.25" extent="1-16" drill="0.5"/>
 <polygon width="0.254" layer="1" thermals="no">
-<vertex x="88" y="43.75"/>
+<vertex x="87.75" y="43.75"/>
 <vertex x="91.5" y="43.75"/>
 <vertex x="91.5" y="35"/>
-<vertex x="88" y="35"/>
+<vertex x="87.75" y="35"/>
 </polygon>
 <wire x1="71" y1="39.15" x2="70.6564" y2="38.8064" width="0.4064" layer="1"/>
@@
 <via x="65.75" y="2.5" extent="1-16" drill="0.5"/>
 <polygon width="0.4064" layer="1" thermals="no">
-<vertex x="60.75" y="4.5"/>
+<vertex x="60.75" y="5"/>
 <vertex x="60.75" y="0.5"/>
 <vertex x="66.75" y="0.5"/>
-<vertex x="66.75" y="4.5"/>
+<vertex x="66.75" y="5"/>
 </polygon>
 <via x="73" y="44.5" extent="1-16" drill="0.5"/>
@@
 <via x="13" y="66.5" extent="1-16" drill="0.5"/>
 <contactref element="J1" pad="2"/>
+<via x="65.75" y="3.75" extent="1-16" drill="0.5"/>
 <wire x1="59.0882" y1="37.9936" x2="59.0882" y2="39.5938" width="0" layer="19" extent="1-1"/>
+<via x="64.25" y="3.75" extent="1-16" drill="0.5"/>
 </signal>
 <signal name="BATT+">
