File: Layout/v1/early-bird.sch (EAGLE design)
At the start: 28 parts, among them U1 ATMEGA328P-AU

Commit message: Add PCB progress.
Parts:
- added C11, C16, C22: 1uF, resistor:C-EUC0603
- added C12, C17, C18, C21: 100n, resistor:C-EUC0402
- added C13: 10uF, resistor:C-EUC1210
- added C14, C15: 22p, resistor:C-EUC0402
- added C19: 33n, resistor:C-EUC0402
- added C20: (no value), resistor:C-EUC0402
- added D1: MBRA340T3, diode:MBRA340T3
- added J1: 22-27-2021-02, con-molex:22-27-2021-02
- added J2: AVR_SPI_PRG_62X3_LOCK, SparkFun-Connectors:AVR_SPI_PRG_62X3_LOCK
- added JP1: M02PTH, SparkFun-Connectors:M02PTH
- added LED4: (no value), led:LEDCHIPLED_1206
- added R10, R7, R8, R9: 10, resistor:R-EU_R0402
- added R11, R12, R13, R14: (no value), resistor:R-EU_R0402
- added U$10: MULTICOMP_8MM_INDUCTOR, Ava:MULTICOMP_8MM_INDUCTOR
- added U$7: ABRACON_ABM3_CRYSTAL, Ava:ABRACON_ABM3_CRYSTAL
- added U$8: ADP1612, Ava:ADP1612
- added U$9: BGM1034N7, Ava:BGM1034N7
- C9: value 100n -> 10uF; device resistor:C-EUC0402 -> resistor:C-EUC1210
- U$1, U$2: value KEYSTONE-82-AAA-BATTERY-HOLDER -> KEYSTONE-92-AA-BATTERY-HOLDER; device Ava:KEYSTONE-82-AAA-BATTERY-HOLDER -> Ava:KEYSTONE-92-AA-BATTERY-HOLDER
Connections:
- removed net +: C2.1, C3.1, C4.1, C5.1, C6.1, C7.1, R1.2, R2.2, R4.1, U$4.VCC, U$5.6_V_BCKP, U$5.7_VCC_IO, U$5.8_VCC, U1.AVCC, U1.VCC, U1.VCC_2
- removed net -: C1.2, C10.2, C2.2, C3.2, C4.2, C5.2, C6.2, C7.2, C8.2, C9.2, LED1.C, LED2.C, LED3.C, R3.1, U$4.GND@1, U$4.GND@2, U$4.GND@3, U$5.10_GND, U$5.12_GND, U$5.1_GND, U$6.GND, U1.GND, U1.GND_2, U1.GND_3
- removed net N$9: U$4.DIO0
- new net AUX+: C11.1, C12.1, C13.1, D1.C, J1-1.S, R10.1, R13.2
- new net BATT+: C16.1, C17.1, C18.1, C2.1, C21.1, C22.1, C3.1, C4.1, C5.1, C6.1, C7.1, C9.1, J2.2, JP1.1, JP1.2, R1.2, R14.2, R2.2, R4.1, U$1.BATT+, U$10.P$2, U$4.VCC, U$5.6_V_BCKP, U$5.7_VCC_IO, U$5.8_VCC, U$8.EN, U$8.VIN, U1.AVCC, U1.VCC, U1.VCC_2
- new net BATT-: C1.2, C10.2, C11.2, C12.2, C13.2, C14.2, C15.2, C16.2, C17.2, C18.2, C19.2, C2.2, C20.1, C21.2, C22.2, C3.2, C4.2, C5.2, C6.2, C7.2, C8.2, C9.2, J1-2.S, J2.6, L1.2, LED1.C, LED2.C, LED3.C, LED4.C, R12.1, R14.1, R3.1, U$2.BATT-, U$4.GND@1, U$4.GND@2, U$4.GND@3, U$5.10_GND, U$5.12_GND, U$5.1_GND, U$6.GND, U$8.FREQ, U$8.GND, U$9.GND, U1.GND, U1.GND_2, U1.GND_3
- new net DIO0: U$4.DIO0, U1.PD7
- new net DIO1: U$4.DIO1, U1.PB0
- new net DIO2: U$4.DIO2, U1.PB1
- new net LNA+: C10.1, R4.2, U$9.PON, U$9.VCC
- new net N$10: R7.1, U1.PD2
- new net N$12: R8.1, U1.PD3
- new net N$13: R9.1, U1.PD4
- new net N$14: LED1.A, R9.2
- new net N$15: LED4.A, R10.2
- new net N$16: U$1.BATT-, U$2.BATT+
- new net N$17: C15.1, U$7.2, U1.PB7
- new net N$18: C14.1, U$7.1, U1.PB6
- new net N$19: C19.1, U$8.SS
- new net N$20: R11.2, U$8.COMP
- new net N$21: R12.2, R13.1, U$8.FB
- new net N$23: D1.A, U$10.P$1, U$8.SW
- new net N$24: L2.2, U$9.AI
- new net N$25: U$5.11_RF_IN, U$9.RFOUT
- net MISO: now also J2.1
- net MOSI: now also J2.4
- net N$11: now also L2.1, U$9.SO; no longer C10.1, C9.1, R4.2
- net N$2: now also L1.1, U$9.RFIN; no longer U$5.11_RF_IN
- net N$3: now also LED3.A, R7.2; no longer LED1.A, U1.PD2
- net N$4: now also R8.2; no longer U1.PD3
- net N$5: now also C20.2, R11.1; no longer LED3.A, U1.PD4
- net RESET: now also J2.5
- net SCK: now also J2.3
Other:
- moved on the sheet: C1, C9, L1, L2

Commit message: Layout Progress, redraw schematic a little.
Parts:
- added C23: 10uF, resistor:C-EUC1210
Connections:
- new net N$9: JP1.1, R14.2, U$8.EN
- net BATT+: now also C23.1; no longer JP1.1, R14.2, U$8.EN
- net BATT-: now also C23.2
Other:
- moved on the sheet: C10, L2, R4
Changed lines of the file:
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@@
 <part name="C9" library="resistor" deviceset="C-EU" device="C1210" value="10uF"/>
 <part name="R14" library="resistor" deviceset="R-EU_" device="R0402"/>
+<part name="C23" library="resistor" deviceset="C-EU" device="C1210" value="10uF"/>
 </parts>
 <sheets>
@@
 <instance part="C8" gate="G$1" x="33.02" y="27.94"/>
 <instance part="L1" gate="G$1" x="68.58" y="124.46"/>
-<instance part="L2" gate="G$1" x="88.9" y="152.4" rot="R90"/>
+<instance part="L2" gate="G$1" x="88.9" y="154.94" rot="R90"/>
 <instance part="C5" gate="G$1" x="12.7" y="63.5"/>
 <instance part="C6" gate="G$1" x="22.86" y="63.5"/>
 <instance part="C7" gate="G$1" x="33.02" y="63.5"/>
-<instance part="C10" gate="G$1" x="50.8" y="134.62"/>
-<instance part="R4" gate="G$1" x="33.02" y="139.7"/>
+<instance part="C10" gate="G$1" x="114.3" y="149.86"/>
+<instance part="R4" gate="G$1" x="142.24" y="154.94" rot="R180"/>
 <instance part="R5" gate="G$1" x="185.42" y="106.68"/>
 <instance part="R6" gate="G$1" x="185.42" y="101.6"/>
@@
 <instance part="C9" gate="G$1" x="-66.04" y="-33.02"/>
 <instance part="R14" gate="G$1" x="-22.86" y="-40.64" rot="R90"/>
+<instance part="C23" gate="G$1" x="55.88" y="63.5"/>
 </instances>
 <busses>
@@
 <junction x="35.56" y="55.88"/>
 <label x="15.24" y="55.88" size="1.778" layer="95"/>
+<pinref part="C23" gate="G$1" pin="2"/>
+<wire x1="40.64" y1="55.88" x2="55.88" y2="55.88" width="0.1524" layer="91"/>
+<wire x1="55.88" y1="55.88" x2="55.88" y2="58.42" width="0.1524" layer="91"/>
+<junction x="40.64" y="55.88"/>
 </segment>
 <segment>
@@
 <segment>
 <pinref part="C10" gate="G$1" pin="2"/>
-<wire x1="40.64" y1="127" x2="50.8" y2="127" width="0.1524" layer="91"/>
-<wire x1="50.8" y1="127" x2="50.8" y2="129.54" width="0.1524" layer="91"/>
-<label x="43.18" y="127" size="1.778" layer="95"/>
+<wire x1="114.3" y1="142.24" x2="114.3" y2="144.78" width="0.1524" layer="91"/>
+<label x="116.84" y="142.24" size="1.778" layer="95"/>
+<wire x1="114.3" y1="142.24" x2="124.46" y2="142.24" width="0.1524" layer="91"/>
 </segment>
 <segment>
@@
 <junction x="35.56" y="68.58"/>
 <label x="15.24" y="68.58" size="1.778" layer="95"/>
-</segment>
-<segment>
+<pinref part="C23" gate="G$1" pin="1"/>
+<wire x1="40.64" y1="68.58" x2="55.88" y2="68.58" width="0.1524" layer="91"/>
+<wire x1="55.88" y1="68.58" x2="55.88" y2="66.04" width="0.1524" layer="91"/>
+<junction x="40.64" y="68.58"/>
+</segment>
+<segment>
+<pinref part="R2" gate="G$1" pin="2"/>
+<wire x1="25.4" y1="45.72" x2="15.24" y2="45.72" width="0.1524" layer="91"/>
+<label x="15.24" y="45.72" size="1.778" layer="95"/>
+</segment>
+<segment>
+<pinref part="R4" gate="G$1" pin="1"/>
+<wire x1="147.32" y1="154.94" x2="177.8" y2="154.94" width="0.1524" layer="91"/>
+<label x="185.42" y="132.08" size="1.778" layer="95"/>
 <pinref part="U$5" gate="G$1" pin="8_VCC"/>
 <wire x1="175.26" y1="132.08" x2="177.8" y2="132.08" width="0.1524" layer="91"/>
@@
 <wire x1="177.8" y1="121.92" x2="177.8" y2="127" width="0.1524" layer="91"/>
 <junction x="177.8" y="127"/>
-</segment>
-<segment>
-<pinref part="R2" gate="G$1" pin="2"/>
-<wire x1="25.4" y1="45.72" x2="15.24" y2="45.72" width="0.1524" layer="91"/>
-<label x="15.24" y="45.72" size="1.778" layer="95"/>
-</segment>
-<segment>
-<pinref part="R4" gate="G$1" pin="1"/>
-<wire x1="27.94" y1="139.7" x2="22.86" y2="139.7" width="0.1524" layer="91"/>
-<label x="20.32" y="139.7" size="1.778" layer="95"/>
+<wire x1="177.8" y1="154.94" x2="177.8" y2="132.08" width="0.1524" layer="91"/>
 </segment>
 <segment>
@@
 <wire x1="-20.32" y1="-27.94" x2="-20.32" y2="-22.86" width="0.1524" layer="91"/>
 <junction x="-20.32" y="-22.86"/>
-<pinref part="U$8" gate="G$1" pin="EN"/>
-<pinref part="JP1" gate="G$1" pin="1"/>
-<wire x1="-10.16" y1="-30.48" x2="-17.78" y2="-30.48" width="0.1524" layer="91"/>
-<wire x1="-17.78" y1="-30.48" x2="-22.86" y2="-30.48" width="0.1524" layer="91"/>
-<wire x1="-20.32" y1="-27.94" x2="-17.78" y2="-27.94" width="0.1524" layer="91"/>
-<wire x1="-17.78" y1="-27.94" x2="-17.78" y2="-30.48" width="0.1524" layer="91"/>
-<junction x="-20.32" y="-27.94"/>
-<junction x="-17.78" y="-30.48"/>
 <pinref part="U$10" gate="G$1" pin="P$2"/>
 <wire x1="-10.16" y1="-12.7" x2="-12.7" y2="-12.7" width="0.1524" layer="91"/>
@@
 <junction x="-66.04" y="-22.86"/>
 <junction x="-53.34" y="-22.86"/>
-<pinref part="R14" gate="G$1" pin="2"/>
-<wire x1="-22.86" y1="-35.56" x2="-22.86" y2="-30.48" width="0.1524" layer="91"/>
-<junction x="-22.86" y="-30.48"/>
 </segment>
 </net>
@@
 <pinref part="R4" gate="G$1" pin="2"/>
 <pinref part="C10" gate="G$1" pin="1"/>
-<wire x1="38.1" y1="139.7" x2="50.8" y2="139.7" width="0.1524" layer="91"/>
-<wire x1="50.8" y1="139.7" x2="50.8" y2="137.16" width="0.1524" layer="91"/>
-<label x="43.18" y="139.7" size="1.778" layer="95"/>
-</segment>
-<segment>
+<wire x1="137.16" y1="154.94" x2="114.3" y2="154.94" width="0.1524" layer="91"/>
+<wire x1="114.3" y1="154.94" x2="114.3" y2="152.4" width="0.1524" layer="91"/>
 <pinref part="U$9" gate="G$1" pin="PON"/>
-<wire x1="99.06" y1="144.78" x2="99.06" y2="147.32" width="0.1524" layer="91"/>
-<wire x1="99.06" y1="147.32" x2="106.68" y2="147.32" width="0.1524" layer="91"/>
+<wire x1="99.06" y1="144.78" x2="99.06" y2="154.94" width="0.1524" layer="91"/>
+<wire x1="99.06" y1="154.94" x2="106.68" y2="154.94" width="0.1524" layer="91"/>
 <pinref part="U$9" gate="G$1" pin="VCC"/>
-<wire x1="106.68" y1="147.32" x2="106.68" y2="144.78" width="0.1524" layer="91"/>
-<wire x1="106.68" y1="147.32" x2="119.38" y2="147.32" width="0.1524" layer="91"/>
-<junction x="106.68" y="147.32"/>
-<label x="111.76" y="147.32" size="1.778" layer="95"/>
+<wire x1="106.68" y1="154.94" x2="106.68" y2="144.78" width="0.1524" layer="91"/>
+<wire x1="106.68" y1="154.94" x2="114.3" y2="154.94" width="0.1524" layer="91"/>
+<junction x="106.68" y="154.94"/>
+<label x="116.84" y="154.94" size="1.778" layer="95"/>
+<junction x="114.3" y="154.94"/>
 </segment>
 </net>
@@
 <pinref part="L2" gate="G$1" pin="1"/>
 <pinref part="U$9" gate="G$1" pin="SO"/>
-<wire x1="83.82" y1="152.4" x2="83.82" y2="144.78" width="0.1524" layer="91"/>
+<wire x1="83.82" y1="154.94" x2="83.82" y2="144.78" width="0.1524" layer="91"/>
 </segment>
 </net>
@@
 <pinref part="L2" gate="G$1" pin="2"/>
 <pinref part="U$9" gate="G$1" pin="AI"/>
-<wire x1="93.98" y1="152.4" x2="93.98" y2="144.78" width="0.1524" layer="91"/>
+<wire x1="93.98" y1="154.94" x2="93.98" y2="144.78" width="0.1524" layer="91"/>
 </segment>
 </net>
@@
 </segment>
 </net>
+<net name="N$9" class="0">
+<segment>
+<pinref part="JP1" gate="G$1" pin="1"/>
+<pinref part="R14" gate="G$1" pin="2"/>
+<wire x1="-22.86" y1="-35.56" x2="-22.86" y2="-30.48" width="0.1524" layer="91"/>
+<junction x="-22.86" y="-30.48"/>
+<pinref part="U$8" gate="G$1" pin="EN"/>
+<wire x1="-10.16" y1="-30.48" x2="-22.86" y2="-30.48" width="0.1524" layer="91"/>
+</segment>
+</net>

Commit message: Stage for fab?
Parts:
- added PAD1, PAD2: (no value), wirepad:SMD2
- added Q1: (no value), crystal:CRYSTALCTS406
Connections:
- new net N$22: PAD1.P, Q1.1
- new net N$26: PAD2.P, Q1.2
- net BATT-: now also Q1.P$1
Changed lines of the file:
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@@
 <part name="R14" library="resistor" deviceset="R-EU_" device="R0402"/>
 <part name="C23" library="resistor" deviceset="C-EU" device="C1210" value="10uF"/>
+<part name="PAD1" library="wirepad" deviceset="SMD2" device=""/>
+<part name="PAD2" library="wirepad" deviceset="SMD2" device=""/>
+<part name="Q1" library="crystal" deviceset="CRYSTAL" device="CTS406"/>
 </parts>
 <sheets>
@@
 <instance part="R14" gate="G$1" x="-22.86" y="-40.64" rot="R90"/>
 <instance part="C23" gate="G$1" x="55.88" y="63.5"/>
+<instance part="PAD1" gate="1" x="195.58" y="-22.86" rot="R270"/>
+<instance part="PAD2" gate="1" x="205.74" y="-22.86" rot="R270"/>
+<instance part="Q1" gate="G$1" x="200.66" y="-33.02"/>
 </instances>
 <busses>
@@
 <wire x1="226.06" y1="30.48" x2="241.3" y2="30.48" width="0.1524" layer="91"/>
 </segment>
+<segment>
+<pinref part="Q1" gate="G$1" pin="P$1"/>
+<wire x1="200.66" y1="-38.1" x2="200.66" y2="-40.64" width="0.1524" layer="91"/>
+<wire x1="200.66" y1="-40.64" x2="210.82" y2="-40.64" width="0.1524" layer="91"/>
+<label x="205.74" y="-40.64" size="1.778" layer="95"/>
+</segment>
 </net>
 <net name="BATT+" class="0">
@@
 </segment>
 </net>
+<net name="N$22" class="0">
+<segment>
+<pinref part="PAD1" gate="1" pin="P"/>
+<wire x1="195.58" y1="-25.4" x2="195.58" y2="-33.02" width="0.1524" layer="91"/>
+<pinref part="Q1" gate="G$1" pin="1"/>
+<wire x1="195.58" y1="-33.02" x2="198.12" y2="-33.02" width="0.1524" layer="91"/>
+</segment>
+</net>
+<net name="N$26" class="0">
+<segment>
+<pinref part="Q1" gate="G$1" pin="2"/>
+<pinref part="PAD2" gate="1" pin="P"/>
+<wire x1="203.2" y1="-33.02" x2="205.74" y2="-33.02" width="0.1524" layer="91"/>
+<wire x1="205.74" y1="-33.02" x2="205.74" y2="-25.4" width="0.1524" layer="91"/>
+</segment>
+</net>
